File: Starpex Peak PCB.kicad_sch (KiCad schematic)
At the start: 0 parts

Commit message: Peak PCB 1.0
All traces ready. Now need to make daughterboard for RPi Pico
Parts:
- added J1: Conn_01x12_Pin, Custom Footprints:GH, symbol Connector:Conn_01x12_Pin
- added J2: Conn_01x20_Pin, Connector_PinHeader_2.54mm:PinHeader_2x10_P2.54mm_Vertical, symbol Connector:Conn_01x20_Pin
- added SW1: SW_SPDT_321, Custom Footprints:KW11, symbol Switch:SW_SPDT_321
- added SW2, SW3: SW_Push, PCM_Switch_Keyboard_Alps_Matias:SW_Alps_Matias, symbol Switch:SW_Push
Connections:
- new net: J1.1 (Pin_1), J2.2 (Pin_2), SW1.1 (C), SW2.2
- new net: J1.10 (Pin_10), J2.16 (Pin_16)
- new net: J1.11 (Pin_11), J2.14 (Pin_14)
- new net: J1.12 (Pin_12), J2.12 (Pin_12)
- new net: J1.2 (Pin_2), J2.3 (Pin_3)
- new net: J1.3 (Pin_3), J2.5 (Pin_5)
- new net: J1.4 (Pin_4), J2.7 (Pin_7)
- new net: J1.5 (Pin_5), J2.9 (Pin_9)
- new net: J1.6 (Pin_6), J2.13 (Pin_13)
- new net: J1.7 (Pin_7), J2.17 (Pin_17)
- new net: J1.8 (Pin_8), J2.19 (Pin_19)
- new net: J1.9 (Pin_9), J2.20 (Pin_20)
- new net: J2.11 (Pin_11), SW3.1
- new net: J2.15 (Pin_15), SW3.2
- new net: J2.4 (Pin_4), SW2.1
- new net: J2.6 (Pin_6), SW1.2 (B)
