File: Starpex Peak PCB.kicad_sch (KiCad schematic)
At the start: 5 parts, among them J1 Conn_01x12_Pin, J2 Conn_01x20_Pin, SW1 SW_SPDT_321, SW2 SW_Push, SW3 SW_Push

Commit message: help from Vincent Santosa
with the old DuPont connector design
Connections:
- net GND: now reaches J1.1 (Pin_1), J2.2 (Pin_2), SW2.2
- net GND: now also J1.12 (Pin_12), SW1.2 (B), SW3.2; no longer SW1.1 (C)
- net at J2.16 (Pin_16): no longer J1.10 (Pin_10)
- net at J2.14 (Pin_14): no longer J1.11 (Pin_11)
- net at J2.12 (Pin_12): no longer J1.12 (Pin_12)
- net 1: now reaches J1.2 (Pin_2)
- net 1: now also J2.1 (Pin_1); no longer J2.3 (Pin_3)
- net 2: now reaches J1.3 (Pin_3)
- net 2: now also J2.3 (Pin_3); no longer J2.5 (Pin_5)
- net 3: now reaches J1.4 (Pin_4)
- net 3: now also J2.5 (Pin_5); no longer J2.7 (Pin_7)
- net 4: now reaches J1.5 (Pin_5)
- net 4: now also J2.7 (Pin_7); no longer J2.9 (Pin_9)
- net 5: now reaches J1.6 (Pin_6)
- net 5: now also J2.9 (Pin_9); no longer J2.13 (Pin_13)
- net 6: now reaches J1.7 (Pin_7)
- net 6: now also J2.11 (Pin_11); no longer J2.17 (Pin_17)
- net 10: now reaches J2.19 (Pin_19)
- net 10: now also J1.11 (Pin_11); no longer J1.8 (Pin_8)
- net 8: now reaches J1.9 (Pin_9)
- net 8: now also J2.15 (Pin_15); no longer J2.20 (Pin_20)
- net B1: now reaches SW3.1
- net B1: now also J2.20 (Pin_20); no longer J2.11 (Pin_11)
- net B2: now reaches J2.4 (Pin_4), SW2.1
- net B3: now reaches J2.6 (Pin_6)
- net B3: now also SW1.3 (A); no longer SW1.2 (B)
- new net 7: J1.8 (Pin_8), J2.13 (Pin_13)
- new net 9: J1.10 (Pin_10), J2.17 (Pin_17)
Other:
- moved on the sheet: J1, SW1, SW2, SW3
